File: catfeeder.kicad_pcb (KiCad board)
At the start: 2 copper layers, 40.1 x 66.9 mm, 88 parts, among them J1 Barrel_Jack_Switch, J2 USB_B_Mini, J3 RFID, J4 DoorOpen, J5 Scale, J6 Auger Motor, J7 Door Motor, J8 DoorClose, M1 Mount, M2 Mount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

Commit message: Cleanup tracks and vias.
Parts:
- L2: moved to F.Cu
- moved L2 4.08 mm to (85.2, 121.2), turned to 180 degrees
- moved C20 1.19 mm to (86.6, 128.0), turned to -90 degrees
- moved C21 0.61 mm to (88.6, 119.0), turned to 180 degrees
Routing:
- net Net-(Q3-C): track 14.7 -> 9.70 mm, vias 2 -> 1
- net /DATA_1: track 22.9 -> 19.7 mm, vias 2 -> 0
- net Net-(J5-Pin_1): track 5.19 -> 7.69 mm
- net /M1_DIR: track 25.8 -> 24.7 mm
- net /M1_SLEEP: track 46.0 -> 45.4 mm
- net /Scale_Rate: track 14.8 -> 14.2 mm, vias 3 -> 1
- net /DATA_0: track 16.8 -> 17.3 mm
